File: IKe.kicad_sch (KiCad schematic)
At the start: 23 parts, among them SW1 SW_SPST, U1 LM741, U11 74HC04, U2 ADS1110, U3 LM741, U4 AD5693RxRM, U5 DRV8847SPWR, U6 ADuM1250, U7 4027, U8 ICE40HX4K-TQ144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

Commit message: Add files via upload
Other:
- note added: "Comparator (1-BIT ADC)"
- note added: "MCU/FPGA/Output"
- note removed: "Comparator"
- note removed: "MCU/FPGA"
Changed lines of the file:
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@@
     (stroke (width 0) (type default))
   )
-  (text "Comparator\n" (at 133.35 50.8 0)
+  (text "Comparator\n(1-BIT ADC)\n" (at 130.81 52.07 0)
     (effects (font (size 1.27 1.27)) (justify left bottom))
   )
@@
     (effects (font (size 1.27 1.27)) (justify left bottom))
   )
-  (text "MCU/FPGA\n" (at 173.99 60.96 0)
+  (text "MCU/FPGA/Output\n" (at 173.99 60.96 0)
     (effects (font (size 1.27 1.27)) (justify left bottom))
   )
